File: tests/fixtures/mixed_symbols.kicad_sch (KiCad schematic)
At the start: 15 parts, among them Q1 NPN, Q2 PNP, Q3 BF244A, Q4 BF545B, SW1 SW_DPST_x2, T1 Transformer_1P_1S, U1 OP1177AR

Commit message: Revert "Centre JFET gate leads on the channel, as KiCad draws them"
This reverts commit db677e2c4029a2e2f560439100e40cadad8258a5.
Parts:
- removed Q4: BF545B, Package_TO_SOT_SMD:SOT-23, symbol Transistor_FET:BF545B
Other:
- moved on the sheet: Q3
Changed lines of the file:
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@@
 	(paper "A4")
 	(junction
-		(at 129.54 144.78)
-		(diameter 0)
-		(color 0 0 0 0)
-	)
-	(junction
 		(at 105.41 90.17)
 		(diameter 0)
@@
 	)
 	(junction
-		(at 133.35 140.97)
-		(diameter 0)
-		(color 0 0 0 0)
-	)
-	(junction
 		(at 115.57 90.17)
 		(diameter 0)
@@
 	)
 	(junction
-		(at 144.78 140.97)
+		(at 133.35 144.78)
 		(diameter 0)
 		(color 0 0 0 0)
@@
 	)
 	(junction
+		(at 148.59 120.65)
+		(diameter 0)
+		(color 0 0 0 0)
+	)
+	(junction
 		(at 133.35 127)
 		(diameter 0)
@@
 	)
 	(junction
-		(at 135.89 140.97)
-		(diameter 0)
-		(color 0 0 0 0)
-	)
-	(junction
 		(at 105.41 107.95)
 		(diameter 0)
@@
 	)
 	(junction
-		(at 151.13 120.65)
-		(diameter 0)
-		(color 0 0 0 0)
-	)
-	(junction
 		(at 128.27 102.87)
 		(diameter 0)
@@
 	)
 	(junction
+		(at 140.97 127)
+		(diameter 0)
+		(color 0 0 0 0)
+	)
+	(junction
 		(at 88.9 107.95)
 		(diameter 0)
@@
 	)
 	(junction
-		(at 143.51 127)
-		(diameter 0)
-		(color 0 0 0 0)
-	)
-	(junction
 		(at 107.95 90.17)
 		(diameter 0)
@@
 	(wire
 		(pts
-			(xy 129.54 144.78) (xy 133.35 144.78)
-		)
-		(stroke
-			(width 0)
-			(type default)
-		)
-	)
-	(wire
-		(pts
 			(xy 102.87 90.17) (xy 105.41 90.17)
 		)
@@
 	(wire
 		(pts
-			(xy 133.35 140.97) (xy 133.35 144.78)
-		)
-		(stroke
-			(width 0)
-			(type default)
-		)
-	)
-	(wire
-		(pts
-			(xy 133.35 127) (xy 143.51 127)
+			(xy 133.35 127) (xy 140.97 127)
 		)
 		(stroke
@@
 	(wire
 		(pts
-			(xy 144.78 152.4) (xy 144.78 154.94)
-		)
-		(stroke
-			(width 0)
-			(type default)
-		)
-	)
-	(wire
-		(pts
 			(xy 105.41 90.17) (xy 105.41 95.25)
 		)
@@
 	(wire
 		(pts
-			(xy 135.89 140.97) (xy 144.78 140.97)
-		)
-		(stroke
-			(width 0)
-			(type default)
-		)
-	)
-	(wire
-		(pts
-			(xy 144.78 140.97) (xy 144.78 142.24)
-		)
-		(stroke
-			(width 0)
-			(type default)
-		)
-	)
-	(wire
-		(pts
 			(xy 88.9 102.87) (xy 88.9 107.95)
 		)
@@
 	(wire
 		(pts
-			(xy 135.89 147.32) (xy 135.89 140.97)
-		)
-		(stroke
-			(width 0)
-			(type default)
-		)
-	)
-	(wire
-		(pts
 			(xy 80.01 102.87) (xy 80.01 107.95)
 		)
@@
 	(wire
 		(pts
-			(xy 144.78 154.94) (xy 129.54 154.94)
-		)
-		(stroke
-			(width 0)
-			(type default)
-		)
-	)
-	(wire
-		(pts
 			(xy 161.29 107.95) (xy 161.29 115.57)
 		)
@@
 	(wire
 		(pts
-			(xy 137.16 147.32) (xy 135.89 147.32)
-		)
-		(stroke
-			(width 0)
-			(type default)
-		)
-	)
-	(wire
-		(pts
 			(xy 128.27 102.87) (xy 153.67 102.87)
 		)
@@
 	(wire
 		(pts
-			(xy 143.51 135.89) (xy 143.51 127)
-		)
-		(stroke
-			(width 0)
-			(type default)
-		)
-	)
-	(wire
-		(pts
-			(xy 125.73 144.78) (xy 129.54 144.78)
+			(xy 140.97 139.7) (xy 140.97 127)
+		)
+		(stroke
+			(width 0)
+			(type default)
+		)
+	)
+	(wire
+		(pts
+			(xy 125.73 144.78) (xy 133.35 144.78)
 		)
 		(stroke
@@
 	(wire
 		(pts
-			(xy 129.54 154.94) (xy 129.54 144.78)
-		)
-		(stroke
-			(width 0)
-			(type default)
-		)
-	)
-	(wire
-		(pts
-			(xy 146.05 120.65) (xy 151.13 120.65)
+			(xy 148.59 120.65) (xy 146.05 120.65)
 		)
 		(stroke
@@
 	(wire
 		(pts
-			(xy 133.35 127) (xy 133.35 140.97)
+			(xy 133.35 127) (xy 133.35 144.78)
 		)
 		(stroke
@@
 	(wire
 		(pts
-			(xy 151.13 120.65) (xy 151.13 130.81)
-		)
-		(stroke
-			(width 0)
-			(type default)
-		)
-	)
-	(wire
-		(pts
-			(xy 143.51 127) (xy 146.05 127)
+			(xy 148.59 120.65) (xy 148.59 134.62)
+		)
+		(stroke
+			(width 0)
+			(type default)
+		)
+	)
+	(wire
+		(pts
+			(xy 140.97 127) (xy 146.05 127)
 		)
 		(stroke
@@
 	(wire
 		(pts
-			(xy 133.35 140.97) (xy 135.89 140.97)
+			(xy 133.35 144.78) (xy 148.59 144.78)
 		)
 		(stroke
@@
 	(wire
 		(pts
-			(xy 144.78 140.97) (xy 151.13 140.97)
-		)
-		(stroke
-			(width 0)
-			(type default)
-		)
-	)
-	(wire
-		(pts
 			(xy 80.01 90.17) (xy 88.9 90.17)
 		)
@@
 	(wire
 		(pts
-			(xy 153.67 120.65) (xy 151.13 120.65)
+			(xy 153.67 120.65) (xy 148.59 120.65)
 		)
 		(stroke
@@
 	)
 	(symbol
-		(lib_id "Transistor_FET:BF545B")
-		(at 142.24 147.32 0)
-		(unit 1)
-		(body_style 1)
-		(exclude_from_sim no)
-		(in_bom yes)
-		(on_board yes)
-		(in_pos_files yes)
-		(dnp no)
-		(fields_autoplaced yes)
-		(property "Reference" "Q4"
-			(at 147.32 146.0499 0)
-			(show_name no)
-			(do_not_autoplace no)
-			(effects
-				(font
-					(size 1.27 1.27)
-				)
-				(justify left)
-			)
-		)
-		(property "Value" "BF545B"
-			(at 147.32 148.5899 0)
-			(show_name no)
-			(do_not_autoplace no)
-			(effects
-				(font
-					(size 1.27 1.27)
-				)
-				(justify left)
-			)
-		)
-		(property "Footprint" "Package_TO_SOT_SMD:SOT-23"
-			(at 147.32 149.225 0)
-			(hide yes)
-			(show_name no)
-			(do_not_autoplace no)
-			(effects
-				(font
-					(size 1.27 1.27)
-					(italic yes)
-				)
-				(justify left)
-			)
-		)
-		(property "Datasheet" "https://www.nxp.com/docs/en/data-sheet/BF545A_BF545B_BF545C.pdf"
-			(at 147.32 151.13 0)
-			(hide yes)
-			(show_name no)
-			(do_not_autoplace no)
-			(effects
-				(font
-					(size 1.27 1.27)
-				)
-				(justify left)
-			)
-		)
-		(property "Description" "15mA Idss, 30V Vgs, N-Channel JFET, SOT-23"
-			(at 142.24 147.32 0)
-			(hide yes)
-			(show_name no)
-			(do_not_autoplace no)
-			(effects
-				(font
-					(size 1.27 1.27)
-				)
-			)
-		)
-		(pin "2"
-		)
-		(pin "3"
-		)
-		(pin "1"
-		)
-		(instances
-			(project "Testing"
-				(path "/339a58e5-d3b3-42c1-934c-33ac2c9bf58f"
-					(reference "Q4")
-					(unit 1)
-				)
-			)
-		)
-	)
-	(symbol
 		(lib_id "Device:R")
 		(at 80.01 99.06 0)
@@
 		(property "Reference" "T1"
 			(at 115.5827 129.54 0)
-			(hide yes)
 			(show_name no)
 			(do_not_autoplace no)
@@
 		(property "Value" "Transformer_1P_1S"
 			(at 115.5827 132.08 0)
-			(hide yes)
 			(show_name no)
 			(do_not_autoplace no)
@@
 	(symbol
 		(lib_id "Transistor_FET:BF244A")
-		(at 148.59 135.89 0)
+		(at 146.05 139.7 0)
 		(unit 1)
 		(body_style 1)
@@
 		(fields_autoplaced yes)
 		(property "Reference" "Q3"
-			(at 153.67 134.6199 0)
+			(at 151.13 138.4299 0)
 			(show_name no)
 			(do_not_autoplace no)
@@
 		)
 		(property "Value" "BF244A"
-			(at 153.67 137.1599 0)
+			(at 151.13 140.9699 0)
 			(show_name no)
 			(do_not_autoplace no)
@@
 		)
 		(property "Footprint" "Package_TO_SOT_THT:TO-92_Inline"
-			(at 153.67 137.795 0)
+			(at 151.13 141.605 0)
 			(hide yes)
 			(show_name no)
@@
 		)
 		(property "Datasheet" "https://media.digikey.com/pdf/Data%20Sheets/Fairchild%20PDFs/BF244x.pdf"
-			(at 153.67 139.7 0)
+			(at 151.13 143.51 0)
 			(hide yes)
 			(show_name no)
@@
 		)
 		(property "Description" "50mA Id, 30V Vgs, N-Channel FET Transistor, TO-92"
-			(at 148.59 135.89 0)
+			(at 146.05 139.7 0)
 			(hide yes)
 			(show_name no)
@@
 		(property "Reference" "SW1"
 			(at 96.52 99.0599 90)
-			(hide yes)
 			(show_name no)
 			(do_not_autoplace no)
@@
 		(property "Value" "SW_DPST_x2"
 			(at 96.52 101.5999 90)
-			(hide yes)
-			(show_name no)
-			(do_not_autoplace no)
+			(show_name no)
+			(do_not_autoplace no)
