File: tests/fixtures/mixed_symbols.kicad_sch (KiCad schematic)
At the start: 20 parts, among them Q1 NPN, Q2 PNP, Q3 BF244A, Q4 BF545B, SW1 SW_DPST_x2, SW2 SW_DPST_x2, T1 Transformer_1P_1S, U1 OP1177AR

Commit message: Render polar-form values and stop dropping symbols silently
V1's value '10<90' (Unicode U+2220) came out as '1090': _escape() drops any
non-ASCII character it has no LaTeX form for, and the angle sign was not in
the map.

- the angle sign now maps to \$\angle\$, along with the other symbols that
  turn up in component values (+/-, x, .., <=, >=, ~=, superscripts, common
  Greek, dashes and curly quotes)
- _unmapped() plus a generator warning report anything still without a
  mapping, so a mangled value can never pass unnoticed again
- format_value() understands polar form ('10<90', '10@90', '10 angle -45')
  and speaks it as '10 Volt at an angle of 90 degrees'; the phase is moved
  after the reference so the sentence reads 'a 10 Volt AC voltage source
  labelled V1 at an angle of 90 degrees'

Fixture refreshed with the phasor source.
Parts:
- added B2: 5A, symbol Independent_Current_Source:Independent_Current_Source
- added I1: 2A, symbol Simulation_SPICE:IDC
- added L1: 2mH, symbol Polarized_L_Test:L_Polarized
- added V1: 10∠90, symbol Simulation_SPICE:VSIN
- added V2: 5V, symbol Simulation_SPICE:VDC
Connections:
- net at T1.2 (AB), U1.2 (-): no longer L4.1
- net at TR1.1: now also V2.1
- net at TR1.4: now also V2.2
- net at C2.2, T1.1 (AA): no longer L2.1
Other:
- moved on the sheet: L2
